Commit message: baselines + everything here

File: resources/objects/lack_table/lack.urdf (robot description, URDF)
Before this commit: robot object, 1 links, 0 joints
Links:
- added link top, mass 0.0; visual box size=0.0 0.0 0.0
Joints:
- added joint top_fixed: type fixed, parent object, child top, origin xyz=0.0 0 0.2 rpy=0 0 0

File: resources/scenes/8903/two_room_house.urdf (robot description, URDF)
Before this commit: robot 8903, 9 links, 8 joints
Links:
- link back_wall: geometry collision box size=6.0 0.1 0.5; visual box size=6.0 0.1 3.0
- link back_wall_2: geometry collision box size=6.0 0.1 0.5; visual box size=6.0 0.1 3.0
- link door_left_wall: geometry collision box size=2.5 0.1 0.5; visual box size=2.5 0.1 3.0
- link door_right_wall: geometry collision box size=2.5 0.1 0.5; visual box size=2.5 0.1 3.0
- link left_wall: geometry collision box size=12.0 0.1 0.5; visual box size=12.0 0.1 3.0
- link right_wall: geometry collision box size=12.0 0.1 0.5; visual box size=12.0 0.1 3.0
