Commit message: fixed success_rate, early term on success

File: resources/objects/couch2/couch.urdf (robot description, URDF)
Before this commit: robot object, 1 links, 0 joints
Links:
- link object: geometry collision mesh filename=mesh/couch_lowpoly.obj; visual mesh filename=mesh/couch_lowpoly.obj

Commit message: randomize gains, save_config

File: resources/objects/couch2/couch.urdf (robot description, URDF)
Before this commit: robot object, 1 links, 0 joints
Links:
- link object: geometry collision mesh filename=mesh/couch_lowpoly.obj; visual mesh filename=mesh/couch_tex.obj
