Commit message: adding ballu env, COM DR to two legged balance

File: resources/robots/a1/urdf/a1_mass_shift.urdf (robot description, URDF)
Before this commit: robot a1_description, 23 links, 22 joints
Links:
- added link back_mass, mass 0.001; collision box size=0.05 0.194 0.01
- added link front_mass, mass 0.001; collision box size=0.05 0.194 0.01
Joints:
- added joint back_fixed: type fixed, parent trunk, child back_mass, origin xyz=-0.1 0 0.07 rpy=0 0 0
- added joint front_fixed: type fixed, parent trunk, child front_mass, origin xyz=0.1 0 0.07 rpy=0 0 0

Commit message: fb

File: resources/robots/a1/urdf/a1_mass_shift.urdf (robot description, URDF)
Before this commit: robot a1_description, 25 links, 24 joints
Links:
- link back_mass: mass 0.001 -> 0.5; geometry 
- link front_mass: mass 0.001 -> 0.5; geometry 
Joints:
- joint back_fixed: origin xyz=-0.1 0 0.07 rpy=0 0 0 -> xyz=-0.1 0 0.0 rpy=0 0 0
- joint front_fixed: origin xyz=0.1 0 0.07 rpy=0 0 0 -> xyz=0.1 0 0.0 rpy=0 0 0
